File: pcb/Frontend.kicad_sch (KiCad schematic)
At the start: 92 parts, among them J1 Conn_02x05_Top_Bottom, J2 Conn_02x05_Top_Bottom, U101 GAQY212GS, U102 GAQY212GS, U103 GAQY212GS, U104 GAQY212GS, U105 GAQY212GS, U106 GAQY212GS, U107 GAQY212GS, U108 GAQY212GS, U201 GAQY212GS, U202 GAQY212GS, U203 GAQY212GS, U204 GAQY212GS, U205 GAQY212GS, U206 GAQY212GS, U207 GAQY212GS, U208 GAQY212GS, U301 GAQY212GS, U302 GAQY212GS, U303 GAQY212GS, U304 GAQY212GS, U305 GAQY212GS, U306 GAQY212GS, U307 GAQY212GS, U308 GAQY212GS, U401 GAQY212GS, U402 GAQY212GS, U403 GAQY212GS, U404 GAQY212GS, U405 GAQY212GS, U406 GAQY212GS, U407 GAQY212GS, U408 GAQY212GS, U501 GAQY212GS, U502 GAQY212GS, U503 GAQY212GS, U504 GAQY212GS, U505 GAQY212GS, U506 GAQY212GS, U507 GAQY212GS, U508 GAQY212GS

Commit message: Functional block routing
Parts:
- removed J1, J2: Conn_02x05_Top_Bottom, Connector_IDC:IDC-Header_2x05_P2.54mm_Vertical, symbol Connector_Generic:Conn_02x05_Odd_Even
- added J701, J702: DA15_Pins_MountingHoles, Connector_Dsub:DSUB-15_Pins_Horizontal_P2.77x2.84mm_EdgePinOffset4.94mm_Housed_MountingHolesOffset4.94mm, symbol Connector:DA15_Pins_MountingHoles
- added R601, R602, R603, R604, R605, R606, R607, R608, R609, R610, R611, R612, R701, R702, R703, R704, R705, R706, R707, R708, R709, R710, R711, R712: 50k, Resistor_SMD:R_0603_1608Metric_Pad0.98x0.95mm_HandSolder, symbol Device:R
- added RN11, RN12, RN13, RN14, RN15, RN16: 470R, Resistor_SMD:R_Array_Convex_4x0603, symbol Device:R_Pack04
- added U601, U602, U603, U604, U605, U606, U607, U608, U609, U610, U611, U612, U701, U702, U703, U704, U705, U706, U707, U708, U709, U710, U711, U712: GAQY212GS, Package_SO:SOP-4_3.8x4.1mm_P2.54mm, symbol Relay_SolidState:CPC1006N
- renumbered R102 to R101, R103 to R102, R104 to R103, R105 to R104, R106 to R105, R107 to R106, R108 to R107, R109 to R108
Connections:
- net +5V: now also R601.1, R602.1, R603.1, R604.1, R605.1, R606.1, R607.1, R608.1, R609.1, R610.1, R611.1, R612.1, R701.1, R702.1, R703.1, R704.1, R705.1, R706.1, R707.1, R708.1, R709.1, R710.1, R711.1, R712.1, U601.1, U602.1, U603.1, U604.1, U605.1, U606.1, U607.1, U608.1, U609.1, U610.1, U611.1, U612.1, U701.1, U702.1, U703.1, U704.1, U705.1, U706.1, U707.1, U708.1, U709.1, U710.1, U711.1, U712.1
- net at U106.3, U206.3, U306.3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: now also J702.11 (P111)
- net at U201.4, U202.4, U203.4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: now also J702.2
- net at U105.3, U205.3, U305.3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: now also J702.10 (P10)
- net at U101.4, U102.4, U103.4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: now also J702.1
- net at U102.3, U202.3, U302.3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: now also J702.7
- net at U501.4, U502.4, U503.4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: now also J702.5
- net at U107.3, U207.3, U307.3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: now also J702.12 (P12)
- net at U101.3, U201.3, U301.3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: now also J702.6
- net at U401.4, U402.4, U403.4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: now also J702.4
- net at U104.3, U204.3, U304.3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: now also J702.9 (P9)
- net at U301.4, U302.4, U303.4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: now also J702.3
- net at U103.3, U203.3, U303.3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: now also J702.8
- net at U108.3, U208.3, U308.3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: now also J702.13 (P13)
- new net: J701.14 (P14), U612.3, U712.3
- new net: J701.2, U701.4, U702.4, U703.4, U704.4, U705.4, U706.4, U707.4, U708.4, U710.4, U711.4, U712.4
- new net: J701.12 (P12), U610.3, U710.3
- new net: J701.11 (P111), U609.3, U709.3
- new net: J701.10 (P10), U608.3, U708.3
- new net: J701.1, U601.4, U602.4, U603.4, U604.4, U605.4, U606.4, U607.4, U608.4, U610.4, U611.4, U612.4
- new net: J701.13 (P13), U611.3, U711.3
- new net: J701.3, U601.3, U701.3
- new net: J701.4, U602.3, U702.3
- new net: J701.5, U603.3, U703.3
- new net: J701.6, U604.3, U704.3
- new net: J701.7, U605.3, U705.3
- new net: J701.8, U606.3, U706.3
- new net: J701.9 (P9), U607.3, U707.3
- new net 601: R601.2, RN11.5 (R4.2), U601.2
- new net 602: R602.2, RN11.6 (R3.2), U602.2
- new net 603: R603.2, RN11.7 (R2.2), U603.2
- new net 604: R604.2, RN11.8 (R1.2), U604.2
- new net 605: R605.2, RN12.4 (R4.1), U605.2
- new net 606: R606.2, RN12.3 (R3.1), U606.2
- new net 607: R607.2, RN12.2 (R2.1), U607.2
- new net 608: R608.2, RN12.1 (R1.1), U608.2
- new net 609: R609.2, RN13.5 (R4.2), U609.2
- new net 610: R610.2, RN13.6 (R3.2), U610.2
- new net 611: R611.2, RN13.7 (R2.2), U611.2
- new net 612: R612.2, RN13.8 (R1.2), U612.2
- new net 701: R701.2, RN14.4 (R4.1), U701.2
- new net 702: R702.2, RN14.3 (R3.1), U702.2
- new net 703: R703.2, RN14.2 (R2.1), U703.2
- new net 704: R704.2, RN14.1 (R1.1), U704.2
- new net 705: R705.2, RN15.5 (R4.2), U705.2
- new net 706: R706.2, RN15.6 (R3.2), U706.2
- new net 707: R707.2, RN15.7 (R2.2), U707.2
- new net 708: R708.2, RN15.8 (R1.2), U708.2
- new net 709: R709.2, RN16.4 (R4.1), U709.2
- new net 710: R710.2, RN16.3 (R3.1), U710.2
- new net 711: R711.2, RN16.2 (R2.1), U711.2
- new net 712: R712.2, RN16.1 (R1.1), U712.2
- new net Driver5/Q0: RN11.4 (R4.1)
- new net Driver5/Q1: RN11.3 (R3.1)
- new net Driver5/Q2: RN11.2 (R2.1)
- new net Driver5/Q3: RN11.1 (R1.1)
- new net Driver5/Q4: RN12.5 (R4.2)
- new net Driver5/Q5: RN12.6 (R3.2)
- new net Driver5/Q6: RN12.7 (R2.2)
- new net Driver5/Q7: RN12.8 (R1.2)
- new net Driver6/Q0: RN13.4 (R4.1)
- new net Driver6/Q1: RN13.3 (R3.1)
- new net Driver6/Q2: RN13.2 (R2.1)
- new net Driver6/Q3: RN13.1 (R1.1)
- new net Driver6/Q4: RN14.5 (R4.2)
- new net Driver6/Q5: RN14.6 (R3.2)
- new net Driver6/Q6: RN14.7 (R2.2)
- new net Driver6/Q7: RN14.8 (R1.2)
- new net Driver7/Q0: RN15.4 (R4.1)
- new net Driver7/Q1: RN15.3 (R3.1)
- new net Driver7/Q2: RN15.2 (R2.1)
- new net Driver7/Q3: RN15.1 (R1.1)
- new net Driver7/Q4: RN16.5 (R4.2)
- new net Driver7/Q5: RN16.6 (R3.2)
- new net Driver7/Q6: RN16.7 (R2.2)
- new net Driver7/Q7: RN16.8 (R1.2)
- new net Earth_Protective: J701.0 (PAD), J701.15 (P15), J702.0 (PAD)
Other:
- added sheet Driver5 (driver.kicad_sch)
- added sheet Driver6 (driver.kicad_sch)
- added sheet Driver7 (driver.kicad_sch)
- moved on the sheet: R101, R102, R103, R104, R105, R106, R107, R108, R201, R202, R203, R204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

Commit message: More routing
Parts:
- renumbered J702 to J1, J701 to J2
Connections:
- net Earth_Protective: now also J1.14 (P14), J1.15 (P15)
- net at J2.2, U701.4, U702.4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: now also U709.4
- net at U609.4: now also J2.1, U601.4, U602.4, U603.4, U604.4, U605.4, U606.4, U607.4, U608.4, U610.4, U611.4, U612.4
- no-connect marks 0 -> 1
Changed lines of the file:
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@@
 	)
 	(junction
+		(at 449.58 99.06)
+		(diameter 0)
+		(color 0 0 0 0)
+	)
+	(junction
 		(at 295.91 86.36)
 		(diameter 0)
@@
 	)
 	(junction
+		(at 115.57 247.65)
+		(diameter 0)
+		(color 0 0 0 0)
+	)
+	(junction
 		(at 52.07 271.78)
 		(diameter 0)
@@
 	)
 	(junction
+		(at 440.69 64.77)
+		(diameter 0)
+		(color 0 0 0 0)
+	)
+	(junction
 		(at 266.7 92.71)
 		(diameter 0)
@@
 	)
 	(junction
+		(at 80.01 247.65)
+		(diameter 0)
+		(color 0 0 0 0)
+	)
+	(junction
 		(at 266.7 125.73)
 		(diameter 0)
@@
 		(color 0 0 0 0)
 	)
+	(no_connect
+		(at 511.81 311.15)
+	)
 	(wire
 		(pts
@@
 	(wire
 		(pts
+			(xy 109.22 247.65) (xy 115.57 247.65)
+		)
+		(stroke
+			(width 0)
+			(type default)
+		)
+	)
+	(wire
+		(pts
 			(xy 506.73 222.25) (xy 511.81 222.25)
 		)
@@
 	(wire
 		(pts
+			(xy 440.69 64.77) (xy 440.69 99.06)
+		)
+		(stroke
+			(width 0)
+			(type default)
+		)
+	)
+	(wire
+		(pts
 			(xy 274.32 198.12) (xy 274.32 199.39)
 		)
@@
 	(wire
 		(pts
-			(xy 115.57 231.14) (xy 115.57 264.16)
+			(xy 115.57 231.14) (xy 115.57 247.65)
 		)
 		(stroke
@@
 	(wire
 		(pts
+			(xy 115.57 247.65) (xy 115.57 264.16)
+		)
+		(stroke
+			(width 0)
+			(type default)
+		)
+	)
+	(wire
+		(pts
 			(xy 543.56 109.22) (xy 541.02 109.22)
 		)
@@
 	(wire
 		(pts
-			(xy 80.01 231.14) (xy 80.01 264.16)
+			(xy 80.01 231.14) (xy 80.01 247.65)
 		)
 		(stroke
@@
 	(wire
 		(pts
-			(xy 449.58 97.79) (xy 449.58 100.33)
+			(xy 449.58 97.79) (xy 449.58 99.06)
 		)
 		(stroke
@@
 	(wire
 		(pts
+			(xy 73.66 247.65) (xy 80.01 247.65)
+		)
+		(stroke
+			(width 0)
+			(type default)
+		)
+	)
+	(wire
+		(pts
 			(xy 238.76 82.55) (xy 238.76 83.82)
 		)
@@
 	(wire
 		(pts
+			(xy 440.69 99.06) (xy 449.58 99.06)
+		)
+		(stroke
+			(width 0)
+			(type default)
+		)
+	)
+	(wire
+		(pts
 			(xy 381 92.71) (xy 383.54 92.71)
 		)
@@
 	(wire
 		(pts
+			(xy 441.96 59.69) (xy 440.69 59.69)
+		)
+		(stroke
+			(width 0)
+			(type default)
+		)
+	)
+	(wire
+		(pts
 			(xy 506.73 80.01) (xy 506.73 115.57)
 		)
@@
 	(wire
 		(pts
+			(xy 80.01 247.65) (xy 80.01 264.16)
+		)
+		(stroke
+			(width 0)
+			(type default)
+		)
+	)
+	(wire
+		(pts
 			(xy 506.73 222.25) (xy 506.73 257.81)
 		)
@@
 	(wire
 		(pts
+			(xy 441.96 64.77) (xy 440.69 64.77)
+		)
+		(stroke
+			(width 0)
+			(type default)
+		)
+	)
+	(wire
+		(pts
 			(xy 73.66 176.53) (xy 109.22 176.53)
 		)
@@
 	(wire
 		(pts
+			(xy 440.69 59.69) (xy 440.69 64.77)
+		)
+		(stroke
+			(width 0)
+			(type default)
+		)
+	)
+	(wire
+		(pts
 			(xy 336.55 175.26) (xy 336.55 191.77)
 		)
@@
 	(wire
 		(pts
+			(xy 449.58 99.06) (xy 449.58 100.33)
+		)
+		(stroke
+			(width 0)
+			(type default)
+		)
+	)
+	(wire
+		(pts
 			(xy 381 182.88) (xy 381 180.34)
 		)
@@
 		(dnp no)
 		(fields_autoplaced yes)
-		(property "Reference" "J701"
+		(property "Reference" "J2"
 			(at 163.83 87.6299 0)
 			(effects
@@
 			(project ""
 				(path "/0c4edb77-9bdf-4103-be66-c5eb9940b163/92da3f15-6ca3-419e-9376-1f5f82193d40"
-					(reference "J701")
+					(reference "J2")
 					(unit 1)
 				)
@@
 		(dnp no)
 		(fields_autoplaced yes)
-		(property "Reference" "J702"
+		(property "Reference" "J1"
 			(at 454.66 73.6599 0)
 			(effects
@@
 			(project "SSM_board"
 				(path "/0c4edb77-9bdf-4103-be66-c5eb9940b163/92da3f15-6ca3-419e-9376-1f5f82193d40"
-					(reference "J702")
+					(reference "J1")
 					(unit 1)
 				)
