File: pcb/Frontend.kicad_sch (KiCad schematic)
At the start: 146 parts, among them J1 DA15_Pins_MountingHoles, J2 DA15_Pins_MountingHoles, U101 GAQY212GS, U102 GAQY212GS, U103 GAQY212GS, U104 GAQY212GS, U105 GAQY212GS, U106 GAQY212GS, U107 GAQY212GS, U108 GAQY212GS, U201 GAQY212GS, U202 GAQY212GS, U203 GAQY212GS, U204 GAQY212GS, U205 GAQY212GS, U206 GAQY212GS, U207 GAQY212GS, U208 GAQY212GS, U301 GAQY212GS, U302 GAQY212GS, U303 GAQY212GS, U304 GAQY212GS, U305 GAQY212GS, U306 GAQY212GS, U307 GAQY212GS, U308 GAQY212GS, U401 GAQY212GS, U402 GAQY212GS, U403 GAQY212GS, U404 GAQY212GS, U405 GAQY212GS, U406 GAQY212GS, U407 GAQY212GS, U408 GAQY212GS, U501 GAQY212GS, U502 GAQY212GS, U503 GAQY212GS, U504 GAQY212GS, U505 GAQY212GS, U506 GAQY212GS, U507 GAQY212GS, U508 GAQY212GS, U601 GAQY212GS, U602 GAQY212GS, U603 GAQY212GS, U604 GAQY212GS, U605 GAQY212GS, U606 GAQY212GS, U607 GAQY212GS, U608 GAQY212GS, U609 GAQY212GS, U610 GAQY212GS, U611 GAQY212GS, U612 GAQY212GS, U701 GAQY212GS, U702 GAQY212GS, U703 GAQY212GS, U704 GAQY212GS, U705 GAQY212GS, U706 GAQY212GS, U707 GAQY212GS, U708 GAQY212GS, U709 GAQY212GS, U710 GAQY212GS, U711 GAQY212GS, U712 GAQY212GS

Commit message: Ready for production
Parts:
- J1, J2: now left out of the parts list
- RN1, RN10, RN11, RN12, RN13, RN14, RN15, RN16, RN2, RN3, RN4, RN5, RN6, RN7, RN8, RN9: Manufacturer_Part_Number (none) -> YC164-FR-07470R
- U101, U102, U103, U104, U105, U106, U107, U108, U201, U202, U203, U204, U205, U206, U207, U208, U301, U302, U303, U304, U305, U306, U307, U308, U401, U402, U403, U404, U405, U406, U407, U408, U501, U502, U503, U504, U505, U506, U507, U508, U601, U602, U603, U604, U605, U606, U607, U608, U609, U610, U611, U612, U701, U702, U703, U704, U705, U706, U707, U708, U709, U710, U711, U712: Manufacturer_Part_Number (none) -> GAQY212GS

Commit message: Unify footprints, add via-in-pad DRC rule, regenerate outputs
Parts:
- R101, R102, R103, R104, R105, R106, R107, R108, R201, R202, R203, R204, R205, R206, R207, R208, R301, R302, R303, R304, R305, R306, R307, R308, R401, R402, R403, R404, R405, R406, R407, R408, R501, R502, R503, R504, R505, R506, R507, R508, R601, R602, R603, R604, R605, R606, R607, R608, R609, R610, R611, R612, R701, R702, R703, R704, R705, R706, R707, R708, R709, R710, R711, R712: footprint Resistor_SMD:R_0603_1608Metric_Pad0.98x0.95mm_HandSolder -> Resistor_SMD:R_0603_1608Metric
