File: pcb/driver.kicad_sch (KiCad schematic)
At the start: 4 parts, among them IC1 STPIC6C595TTR

Commit message: Ready for production
Parts:
- FB1: Manufacturer_Part_Number (none) -> WLBD1608HCU101TL
- R1: Manufacturer_Part_Number (none) -> CRCW060310K0FKTABC
Changed lines of the file:
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@@
+			)
+		)
+		(property "Manufacturer_Part_Number" "CRCW060310K0FKTABC"
+			(at 129.54 87.63 0)
+			(effects
+				(font
+					(size 1.27 1.27)
+				)
+				(hide yes)
 			)
 		)
@@
 			)
 		)
-		(property "Manufacturer_Part_Number" ""
-			(at 149.86 60.96 90)
-			(effects
+		(property "Manufacturer_Part_Number" "WLBD1608HCU101TL"
+			(at 149.86 60.96 90)
+			(effects

Commit message: Unify footprints, add via-in-pad DRC rule, regenerate outputs
Parts:
- C1: footprint Capacitor_SMD:C_0603_1608Metric_Pad1.08x0.95mm_HandSolder -> Capacitor_SMD:C_0603_1608Metric
- R1: footprint Resistor_SMD:R_0603_1608Metric_Pad0.98x0.95mm_HandSolder -> Resistor_SMD:R_0603_1608Metric
Changed lines of the file:
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@@
 			)
 		)
-		(property "Footprint" "Resistor_SMD:R_0603_1608Metric_Pad0.98x0.95mm_HandSolder"
+		(property "Footprint" "Resistor_SMD:R_0603_1608Metric"
 			(at 127.762 87.63 90)
 			(hide yes)
@@
 			)
 		)
-		(property "Footprint" "Capacitor_SMD:C_0603_1608Metric_Pad1.08x0.95mm_HandSolder"
+		(property "Footprint" "Capacitor_SMD:C_0603_1608Metric"
 			(at 160.3248 72.39 0)
 			(hide yes)
